Commit message: mock components displayed in rviz

File: swervebot_description/urdf/main.xacro (robot description, xacro)
@@ -1,4 +1,10 @@
 <?xml version="1.0"?>
-<robot xmlns:xacro="http://www.ros.org/wiki/xacro"  name="swervebot">
-        <xacro:include filename="swervebot.xacro"/>
+<robot xmlns:xacro="http://www.ros.org/wiki/xacro" name="swervebot">
+        <!-- Parameters are set from launch file -->
+        <xacro:arg name="use_mock_hardware" default="false" />
+        <xacro:include filename="swervebot_urdf.xacro" />
+        <xacro:include filename="ros2_control.xacro" />
+        <xacro:swervebot_ros2_control
+                name="swervebot"
+                use_mock_hardware="$(arg use_mock_hardware)" />
 </robot>

File: swervebot_description/urdf/swervebot_urdf.xacro (robot description, xacro)
@@ -1,6 +1,6 @@
 <?xml version="1.0"?>
 <robot xmlns:xacro="http://www.ros.org/wiki/xacro">
-	<xacro:include filename="xacro_macro.xacro" />
-	<!-- # set parameters -->
+	<xacro:include filename="swervebot_macro.xacro" />
+	<!-- set parameters -->
 	<xacro:property name="chassis_length" value="0.35" />
 	<xacro:property name="chassis_width" value="0.35" />
@@ -13,7 +13,7 @@
 	<xacro:property name="wheel_length" value="0.02" />
 	<xacro:property name="wheel_mass" value="0.1" />
-	<!-- # base_link -->
+	<!-- base_link -->
 	<link name="base_link" />
-	<!-- # base_footprint link -->
+	<!-- base_footprint link -->
 	<joint name="base_footprint_joint" type="fixed">
 		<parent link="base_link" />
@@ -22,5 +22,5 @@
 	</joint>
 	<link name="base_footprint" />
-	<!-- # chassis link -->
+	<!-- chassis link -->
 	<joint name="chassis_joint" type="fixed">
 		<parent link="base_link" />
@@ -43,167 +43,167 @@
 		<material>Gazebo/Orange</material>
 	</gazebo>
-	<!-- front_left_steer_hub link -->
-	<joint name="front_left_steer_hub_joint" type="continuous">
-		<parent link="base_link" />
-		<child link="front_left_steer_hub_link" />
+	<!-- steering_front_left link -->
+	<joint name="steering_front_left_joint" type="continuous">
+		<parent link="base_link" />
+		<child link="steering_front_left_link" />
 		<origin
 			xyz="${chassis_length/2-caster_hub_radius} ${chassis_width/2-caster_hub_radius} 0" />
 		<axis xyz="0 0 1" />
 	</joint>
-	<xacro:link_generator name="front_left_steer_hub_link" color_name="white"
-		origin_x="0"
-		origin_y="0"
-		origin_z="${-caster_hub_length/2}"
-		mass="${caster_hub_mass}">
-		<cylinder radius="${caster_hub_radius}" length="${caster_hub_length}" />
-		<xacro:inertial_cylinder
-			mass="${caster_hub_mass}"
-			length="${caster_hub_length}"
-			radius="${caster_hub_radius}" />
-	</xacro:link_generator>
-	<gazebo reference="chassis">
-		<material>Gazebo/White</material>
-	</gazebo>
-	<!-- front_left_wheel link -->
-	<joint name="front_left_drive_wheel_joint" type="continuous">
-		<parent link="front_left_steer_hub_link" />
-		<child link="front_left_drive_wheel_link" />
-		<origin xyz="${-caster_hub_radius} 0 ${-caster_hub_length}"
-			rpy="${pi/2} 0 0" />
-		<axis xyz="0 0 1" />
-	</joint>
-	<xacro:link_generator name="front_left_drive_wheel_link" color_name="black"
-		origin_x="0"
-		origin_y="0"
-		origin_z="0"
-		mass="${wheel_mass}">
-		<cylinder radius="${wheel_radius}" length="${wheel_length}" />
-		<xacro:inertial_cylinder
-			mass="${wheel_mass}"
-			length="${wheel_length}"
-			radius="${wheel_radius}" />
-	</xacro:link_generator>
-	<gazebo reference="chassis">
-		<material>Gazebo/Black</material>
-	</gazebo>
-	<!-- front_right_steer_hub link -->
-	<joint name="front_right_steer_hub_joint" type="continuous">
-		<parent link="base_link" />
-		<child link="front_right_steer_hub_link" />
+	<xacro:link_generator name="steering_front_left_link" color_name="white"
+		origin_x="0"
+		origin_y="0"
+		origin_z="${-caster_hub_length/2}"
+		mass="${caster_hub_mass}">
+		<cylinder radius="${caster_hub_radius}" length="${caster_hub_length}" />
+		<xacro:inertial_cylinder
+			mass="${caster_hub_mass}"
+			length="${caster_hub_length}"
+			radius="${caster_hub_radius}" />
+	</xacro:link_generator>
+	<gazebo reference="chassis">
+		<material>Gazebo/White</material>
+	</gazebo>
+	<!-- driving_front_left link -->
+	<joint name="driving_front_left_joint" type="continuous">
+		<parent link="steering_front_left_link" />
+		<child link="driving_front_left_link" />
+		<origin xyz="${-caster_hub_radius} 0 ${-caster_hub_length}"
+			rpy="${pi/2} 0 0" />
+		<axis xyz="0 0 1" />
+	</joint>
+	<xacro:link_generator name="driving_front_left_link" color_name="black"
+		origin_x="0"
+		origin_y="0"
+		origin_z="0"
+		mass="${wheel_mass}">
+		<cylinder radius="${wheel_radius}" length="${wheel_length}" />
+		<xacro:inertial_cylinder
+			mass="${wheel_mass}"
+			length="${wheel_length}"
+			radius="${wheel_radius}" />
+	</xacro:link_generator>
+	<gazebo reference="chassis">
+		<material>Gazebo/Black</material>
+	</gazebo>
+	<!-- steering_front_right link -->
+	<joint name="steering_front_right_joint" type="continuous">
+		<parent link="base_link" />
+		<child link="steering_front_right_link" />
 		<origin
 			xyz="${chassis_length/2-caster_hub_radius} ${-chassis_width/2+caster_hub_radius} 0" />
 		<axis xyz="0 0 1" />
 	</joint>
-	<xacro:link_generator name="front_right_steer_hub_link" color_name="white"
-		origin_x="0"
-		origin_y="0"
-		origin_z="${-caster_hub_length/2}"
-		mass="${caster_hub_mass}">
-		<cylinder radius="${caster_hub_radius}" length="${caster_hub_length}" />
-		<xacro:inertial_cylinder
-			mass="${caster_hub_mass}"
-			length="${caster_hub_length}"
-			radius="${caster_hub_radius}" />
-	</xacro:link_generator>
-	<gazebo reference="chassis">
-		<material>Gazebo/White</material>
-	</gazebo>
-	<!-- front_right_wheel link -->
-	<joint name="front_right_drive_wheel_joint" type="continuous">
-		<parent link="front_right_steer_hub_link" />
-		<child link="front_right_drive_wheel_link" />
-		<origin xyz="${-caster_hub_radius} 0 ${-caster_hub_length}"
-			rpy="${pi/2} 0 0" />
-		<axis xyz="0 0 1" />
-	</joint>
-	<xacro:link_generator name="front_right_drive_wheel_link" color_name="black"
-		origin_x="0"
-		origin_y="0"
-		origin_z="0"
-		mass="${wheel_mass}">
-		<cylinder radius="${wheel_radius}" length="${wheel_length}" />
-		<xacro:inertial_cylinder
-			mass="${wheel_mass}"
-			length="${wheel_length}"
-			radius="${wheel_radius}" />
-	</xacro:link_generator>
-	<gazebo reference="chassis">
-		<material>Gazebo/Black</material>
-	</gazebo>
-	<!-- back_right_steer_hub link -->
-	<joint name="back_right_steer_hub_joint" type="continuous">
-		<parent link="base_link" />
-		<child link="back_right_steer_hub_link" />
+	<xacro:link_generator name="steering_front_right_link" color_name="white"
+		origin_x="0"
+		origin_y="0"
+		origin_z="${-caster_hub_length/2}"
+		mass="${caster_hub_mass}">
+		<cylinder radius="${caster_hub_radius}" length="${caster_hub_length}" />
+		<xacro:inertial_cylinder
+			mass="${caster_hub_mass}"
+			length="${caster_hub_length}"
+			radius="${caster_hub_radius}" />
+	</xacro:link_generator>
+	<gazebo reference="chassis">
+		<material>Gazebo/White</material>
+	</gazebo>
+	<!-- driving_front_right link -->
+	<joint name="driving_front_right_joint" type="continuous">
+		<parent link="steering_front_right_link" />
+		<child link="driving_front_right_link" />
+		<origin xyz="${-caster_hub_radius} 0 ${-caster_hub_length}"
+			rpy="${pi/2} 0 0" />
+		<axis xyz="0 0 1" />
+	</joint>
+	<xacro:link_generator name="driving_front_right_link" color_name="black"
+		origin_x="0"
+		origin_y="0"
+		origin_z="0"
+		mass="${wheel_mass}">
+		<cylinder radius="${wheel_radius}" length="${wheel_length}" />
+		<xacro:inertial_cylinder
+			mass="${wheel_mass}"
+			length="${wheel_length}"
+			radius="${wheel_radius}" />
+	</xacro:link_generator>
+	<gazebo reference="chassis">
+		<material>Gazebo/Black</material>
+	</gazebo>
+	<!-- steering_rear_right link -->
+	<joint name="steering_rear_right_joint" type="continuous">
+		<parent link="base_link" />
+		<child link="steering_rear_right_link" />
 		<origin
 			xyz="${-chassis_length/2+caster_hub_radius} ${-chassis_width/2+caster_hub_radius} 0" />
 		<axis xyz="0 0 1" />
 	</joint>
-	<xacro:link_generator name="back_right_steer_hub_link" color_name="white"
-		origin_x="0"
-		origin_y="0"
-		origin_z="${-caster_hub_length/2}"
-		mass="${caster_hub_mass}">
-		<cylinder radius="${caster_hub_radius}" length="${caster_hub_length}" />
-		<xacro:inertial_cylinder
-			mass="${caster_hub_mass}"
-			length="${caster_hub_length}"
-			radius="${caster_hub_radius}" />
-	</xacro:link_generator>
-	<gazebo reference="chassis">
-		<material>Gazebo/White</material>
-	</gazebo>
-	<!-- back_right_wheel link -->
-	<joint name="back_right_drive_wheel_joint" type="continuous">
-		<parent link="back_right_steer_hub_link" />
-		<child link="back_right_drive_wheel_link" />
-		<origin xyz="${-caster_hub_radius} 0 ${-caster_hub_length}"
-			rpy="${pi/2} 0 0" />
-		<axis xyz="0 0 1" />
-	</joint>
-	<xacro:link_generator name="back_right_drive_wheel_link" color_name="black"
-		origin_x="0"
-		origin_y="0"
-		origin_z="0"
-		mass="${wheel_mass}">
-		<cylinder radius="${wheel_radius}" length="${wheel_length}" />
-		<xacro:inertial_cylinder
-			mass="${wheel_mass}"
-			length="${wheel_length}"
-			radius="${wheel_radius}" />
-	</xacro:link_generator>
-	<gazebo reference="chassis">
-		<material>Gazebo/Black</material>
-	</gazebo>
-	<!-- back_left_steer_hub link -->
-	<joint name="back_left_steer_hub_joint" type="continuous">
-		<parent link="base_link" />
-		<child link="back_left_steer_hub_link" />
+	<xacro:link_generator name="steering_rear_right_link" color_name="white"
+		origin_x="0"
+		origin_y="0"
+		origin_z="${-caster_hub_length/2}"
+		mass="${caster_hub_mass}">
+		<cylinder radius="${caster_hub_radius}" length="${caster_hub_length}" />
+		<xacro:inertial_cylinder
+			mass="${caster_hub_mass}"
+			length="${caster_hub_length}"
+			radius="${caster_hub_radius}" />
+	</xacro:link_generator>
+	<gazebo reference="chassis">
+		<material>Gazebo/White</material>
+	</gazebo>
+	<!-- driving_rear_right link -->
+	<joint name="driving_rear_right_joint" type="continuous">
+		<parent link="steering_rear_right_link" />
+		<child link="driving_rear_right_link" />
+		<origin xyz="${-caster_hub_radius} 0 ${-caster_hub_length}"
+			rpy="${pi/2} 0 0" />
+		<axis xyz="0 0 1" />
+	</joint>
+	<xacro:link_generator name="driving_rear_right_link" color_name="black"
+		origin_x="0"
+		origin_y="0"
+		origin_z="0"
+		mass="${wheel_mass}">
+		<cylinder radius="${wheel_radius}" length="${wheel_length}" />
+		<xacro:inertial_cylinder
+			mass="${wheel_mass}"
+			length="${wheel_length}"
+			radius="${wheel_radius}" />
+	</xacro:link_generator>
+	<gazebo reference="chassis">
+		<material>Gazebo/Black</material>
+	</gazebo>
+	<!-- steering_rear_left link -->
+	<joint name="steering_rear_left_joint" type="continuous">
+		<parent link="base_link" />
+		<child link="steering_rear_left_link" />
 		<origin
 			xyz="${-chassis_length/2+caster_hub_radius} ${chassis_width/2-caster_hub_radius} 0" />
 		<axis xyz="0 0 1" />
 	</joint>
-	<xacro:link_generator name="back_left_steer_hub_link" color_name="white"
-		origin_x="0"
-		origin_y="0"
-		origin_z="${-caster_hub_length/2}"
-		mass="${caster_hub_mass}">
-		<cylinder radius="${caster_hub_radius}" length="${caster_hub_length}" />
-		<xacro:inertial_cylinder
-			mass="${caster_hub_mass}"
-			length="${caster_hub_length}"
-			radius="${caster_hub_radius}" />
-	</xacro:link_generator>
-	<gazebo reference="chassis">
-		<material>Gazebo/White</material>
-	</gazebo>
-	<!-- back_left_wheel link -->
-	<joint name="back_left_drive_wheel_joint" type="continuous">
-		<parent link="back_left_steer_hub_link" />
-		<child link="back_left_drive_wheel_link" />
-		<origin xyz="${-caster_hub_radius} 0 ${-caster_hub_length}"
-			rpy="${pi/2} 0 0" />
-		<axis xyz="0 0 1" />
-	</joint>
-	<xacro:link_generator name="back_left_drive_wheel_link" color_name="black"
+	<xacro:link_generator name="steering_rear_left_link" color_name="white"
+		origin_x="0"
+		origin_y="0"
+		origin_z="${-caster_hub_length/2}"
+		mass="${caster_hub_mass}">
+		<cylinder radius="${caster_hub_radius}" length="${caster_hub_length}" />
+		<xacro:inertial_cylinder
+			mass="${caster_hub_mass}"
+			length="${caster_hub_length}"
+			radius="${caster_hub_radius}" />
+	</xacro:link_generator>
+	<gazebo reference="chassis">
+		<material>Gazebo/White</material>
+	</gazebo>
+	<!-- driving_rear_left link -->
+	<joint name="driving_rear_left_joint" type="continuous">
+		<parent link="steering_rear_left_link" />
+		<child link="driving_rear_left_link" />
+		<origin xyz="${-caster_hub_radius} 0 ${-caster_hub_length}"
+			rpy="${pi/2} 0 0" />
+		<axis xyz="0 0 1" />
+	</joint>
+	<xacro:link_generator name="driving_rear_left_link" color_name="black"
 		origin_x="0"
 		origin_y="0"
